Commit message: robot arm

File: arm.urdf (robot description, URDF)
Before this commit: robot testarm, 5 links, 4 joints
Links:
- added link arm4, mass 0.040; collision box size=0.010 0.010 0.06; visual box size=0.01 0.01 0.06
- added link gripper1, mass 0.020; collision box size=0.04 0.010 0.010; visual box size=0.04 0.01 0.01
- added link gripper2, mass 0.003; collision box size=0.005 0.010 0.015; visual box size=0.005 0.01 0.015
- added link gripper3, mass 0.003; collision box size=0.005 0.010 0.015; visual box size=0.005 0.01 0.015
- link arm1: mass 0.020 -> 0.040; geometry collision box size=0.010 0.010 0.060; visual box size=0.01 0.01 0.06
- link arm2: mass 0.020 -> 0.040; geometry collision box size=0.010 0.010 0.060; visual box size=0.01 0.01 0.06
- link arm3: mass 0.020 -> 0.040; geometry collision box size=0.010 0.010 0.060; visual box size=0.01 0.01 0.06
- link stand: geometry collision box size=0.03 0.03 0.020; visual box size=0.03 0.03 0.02
Joints:
- added joint arm3_arm4: type revolute, parent arm3, child arm4, origin xyz=0.000 0.000 0.06 rpy=0 0 0, limit lower=-3.15 upper=3.15 effort=10000.0 velocity=0.5
- added joint arm4_gripper1: type fixed, parent arm4, child gripper1, origin xyz=0.000 0.000 0.060 rpy=0 0 0
- added joint gripper1_gripper2: type prismatic, parent gripper1, child gripper2, origin xyz=-0.0175 0.000 0.01 rpy=0 0 0, limit lower=0 upper=0.015 effort=10000.0 velocity=0.5
- added joint gripper1_gripper3: type prismatic, parent gripper1, child gripper3, origin xyz=0.0175 0.000 0.01 rpy=0 0 0, limit lower=-0.015 upper=0 effort=10000.0 velocity=0.5
- joint arm1_arm2: limit lower=-1.57 upper=1.57 effort=10000.0 velocity=0.5 -> lower=-3.15 upper=3.15 effort=10000.0 velocity=0.5; origin xyz=0.000 0.000 0.03 rpy=0 0 0 -> xyz=0.000 0.000 0.06 rpy=0 0 0
- joint arm2_arm3: limit lower=-1.57 upper=1.57 effort=10000.0 velocity=0.5 -> lower=-3.15 upper=3.15 effort=10000.0 velocity=0.5; origin xyz=0.000 0.000 0.03 rpy=0 0 0 -> xyz=0.000 0.000 0.06 rpy=0 0 0
- joint stand_arm1: limit lower=-3.14 upper=3.14 effort=10000.0 velocity=0.5 -> lower=-3.15 upper=3.15 effort=10000.0 velocity=0.5
